File: valve-headphone-amp.kicad_sch (KiCad schematic)
At the start: 52 parts

Commit message: Add LED for glow
Parts:
- added D2: (no value), symbol Device:LED
- added R16: 1k, Resistor_THT:R_Axial_DIN0309_L9.0mm_D3.2mm_P12.70mm_Horizontal, symbol Device:R_US
- C1, C2: value (none) -> 2.2u; footprint (none) -> Capacitor_THT:C_Rect_L7.2mm_W5.5mm_P5.00mm_FKS2_FKP2_MKS2_MKP2
- C3: value (none) -> 1000u; footprint (none) -> w_capacitors:CP_10x20mm_horiz-L
- C4, C5: value (none) -> 100u; footprint (none) -> rubycon:25ZL100MEFCT16.3X11
- C6, C7: value (none) -> 470u; footprint (none) -> Capacitor_THT:CP_Radial_D10.0mm_P5.00mm
- C8: value (none) -> 47u; footprint (none) -> Capacitor_THT:CP_Radial_D5.0mm_P2.50mm
- D1: value (none) -> LED_Dual_AAC; footprint (none) -> LED_THT:LED_D3.0mm-3
- F1: value (none) -> 3JS-2-R; footprint (none) -> fuses:3JS 1-R
- H1, H2, H3, H4, H5: value (none) -> MountingHole_Pad; footprint (none) -> MountingHole:MountingHole_3.2mm_M3_Pad_Via
- HS1, HS2, HS3, HS4: value (none) -> Heatsink; footprint (none) -> heatsink:heatsink_19x13mm
- J1: value (none) -> RCJ-042; footprint (none) -> rca:CUI_RCJ-042
- J2: value (none) -> RCJ-043; footprint (none) -> rca:CUI_RCJ-043
- J3, J7: value (none) -> SJ-435107; footprint (none) -> 3:CUI_SJ-435107
- J4: value (none) -> Conn_01x02; footprint (none) -> Connector_PinHeader_2.54mm:PinHeader_1x02_P2.54mm_Vertical
- J5: value (none) -> PJ-002AH; footprint (none) -> power:CUI_PJ-002AH
- J6: value (none) -> Conn_01x04; footprint (none) -> Connector_PinHeader_2.54mm:PinHeader_1x04_P2.54mm_Vertical
- K1: value (none) -> 6-1462034-7; footprint (none) -> footprints:PC323-12L-X
- Q1, Q2: value (none) -> IRF610; footprint (none) -> Package_TO_SOT_THT:TO-220-3_Horizontal_TabDown
- Q3: value (none) -> SSN1N45; footprint (none) -> Package_TO_SOT_THT:TO-92_Inline_Wide
- R1: value (none) -> 470; footprint (none) -> Resistor_THT:R_Axial_DIN0309_L9.0mm_D3.2mm_P12.70mm_Horizontal
- R10, R11, R12, R13: value (none) -> 1k; footprint (none) -> Resistor_THT:R_Axial_DIN0309_L9.0mm_D3.2mm_P12.70mm_Horizontal
- R14, R2: value (none) -> 240; footprint (none) -> Resistor_THT:R_Axial_DIN0309_L9.0mm_D3.2mm_P12.70mm_Horizontal
- R15: value (none) -> 47k; footprint (none) -> Resistor_THT:R_Axial_DIN0309_L9.0mm_D3.2mm_P12.70mm_Horizontal
- R3: value (none) -> PTR902-1020K-A502; footprint (none) -> pot:TRIM_PTR902-1020K-A502
- R4, R5: value (none) -> 100k; footprint (none) -> Resistor_THT:R_Axial_DIN0309_L9.0mm_D3.2mm_P12.70mm_Horizontal
- R6, R7: value (none) -> 150; footprint (none) -> Resistor_THT:R_Axial_DIN0309_L9.0mm_D3.2mm_P12.70mm_Horizontal
- R8, R9: value (none) -> 10; footprint (none) -> Resistor_THT:R_Axial_DIN0309_L9.0mm_D3.2mm_P12.70mm_Horizontal
- RV1, RV2, RV3: value (none) -> 50k; footprint (none) -> Potentiometer_THT:Potentiometer_Bourns_3296W_Vertical
- U1, U2: value (none) -> LM317_TO-220; footprint (none) -> Package_TO_SOT_THT:TO-220-3_Horizontal_TabDown
- U3: value (none) -> NE555P; footprint (none) -> Package_DIP:DIP-8_W7.62mm
- V1: value (none) -> 12AU7; footprint (none) -> 12au7:socket_gzc9-b
Connections:
- net +12V: now also R16.2
- net GND: now also D2.1 (K)
- new net: D2.2 (A), R16.1

Commit message: update a bit more
Parts:
- removed D2: (no value), symbol Device:LED
- removed R13: 1k, Resistor_THT:R_Axial_DIN0309_L9.0mm_D3.2mm_P12.70mm_Horizontal, symbol Device:R_US
- D1: symbol Device:LED_Dual_AAC -> Device:LED_Dual_AKA
- R15, R16: footprint Resistor_THT:R_Axial_DIN0309_L9.0mm_D3.2mm_P12.70mm_Horizontal -> Resistor_THT:R_Axial_DIN0309_L9.0mm_D3.2mm_P5.08mm_Vertical
Connections:
- net +12V: now also C8.1; no longer R15.1, R16.2
- net GND: now also D1.2 (K), R15.2; no longer C8.2, D1.3 (K)
- net at Q3.2 (G): now also R14.2; no longer R14.1
- net at U3.2 (TR), U3.6 (THR): now also C8.2, R15.1; no longer C8.1, R15.2
- net at R16.1: now also R14.1, U3.3 (Q)
- new net: D1.3 (A2), R16.2
Other:
- moved on the sheet: C8, R14, R15, R16

Commit message: update parts
Parts:
- Q3: value SSN1N45 -> 2N7000; SUPPLIER_URL https://www.digikey.com.au/en/products/detail/onsemi/SSN1N4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 -> https://www.digikey.com.au/en/products/detail/onsemi/2N7000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
- R14, R2: SUPPLIER_URL https://www.digikey.com.au/en/products/detail/vishay-beyschlag-draloric-bc-components/MBA02040C2400FCT00/5062453 -> https://www.digikey.com.au/en/products/detail/vishay-beyschlag-draloric-bc-components/MRS25000C2400FCT00/5064247
- R6, R7: SUPPLIER_URL https://www.digikey.com.au/en/products/detail/vishay-beyschlag-draloric-bc-components/MBA02040C1500FCT00/5062292 -> https://www.digikey.com.au/en/products/detail/vishay-beyschlag-draloric-bc-components/SFR2500001500FR500/595677
- RV1: value 50k -> 5k; SUPPLIER_URL https://www.ebay.com.au/itm/151504157376 -> https://www.ebay.com.au/itm/151504241784
Changed lines of the file:
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@@
       (effects (font (size 1.27 1.27)) hide)
     )
-    (property "SUPPLIER_URL" "https://www.digikey.com.au/en/products/detail/vishay-beyschlag-draloric-bc-components/MBA02040C1500FCT00/5062292" (id 4) (at 102.87 147.955 0)
+    (property "SUPPLIER_URL" "https://www.digikey.com.au/en/products/detail/vishay-beyschlag-draloric-bc-components/SFR2500001500FR500/595677" (id 4) (at 102.87 147.955 0)
       (effects (font (size 1.27 1.27)) hide)
     )
@@
       (effects (font (size 1.27 1.27)) (justify left))
     )
-    (property "Value" "SSN1N45" (id 1) (at 210.6931 108.3822 0)
+    (property "Value" "2N7000" (id 1) (at 210.6931 108.3822 0)
       (effects (font (size 1.27 1.27)) (justify left))
     )
@@
       (effects (font (size 1.27 1.27)) hide)
     )
-    (property "SUPPLIER_URL" "https://www.digikey.com.au/en/products/detail/onsemi/SSN1N45BTA/1052982" (id 5) (at 215.9 106.68 0)
+    (property "SUPPLIER_URL" "https://www.digikey.com.au/en/products/detail/onsemi/2N7000BU/976604" (id 5) (at 215.9 106.68 0)
       (effects (font (size 1.27 1.27)) hide)
     )
@@
       (effects (font (size 1.27 1.27)) hide)
     )
-    (property "SUPPLIER_URL" "https://www.digikey.com.au/en/products/detail/vishay-beyschlag-draloric-bc-components/MBA02040C1500FCT00/5062292" (id 4) (at 102.87 71.12 0)
+    (property "SUPPLIER_URL" "https://www.digikey.com.au/en/products/detail/vishay-beyschlag-draloric-bc-components/SFR2500001500FR500/595677" (id 4) (at 102.87 71.12 0)
       (effects (font (size 1.27 1.27)) hide)
     )
@@
       (effects (font (size 1.27 1.27)) (justify left))
     )
-    (property "Value" "50k" (id 1) (at 52.578 79.8072 90)
+    (property "Value" "5k" (id 1) (at 52.578 79.8072 90)
       (effects (font (size 1.27 1.27)) (justify left))
     )
@@
       (effects (font (size 1.27 1.27)) (justify left bottom) hide)
     )
-    (property "SUPPLIER_URL" "https://www.ebay.com.au/itm/151504157376" (id 8) (at 50.8 78.105 0)
+    (property "SUPPLIER_URL" "https://www.ebay.com.au/itm/151504241784" (id 8) (at 50.8 78.105 0)
       (effects (font (size 1.27 1.27)) hide)
     )
@@
       (effects (font (size 1.27 1.27)) hide)
     )
-    (property "SUPPLIER_URL" "https://www.digikey.com.au/en/products/detail/vishay-beyschlag-draloric-bc-components/MBA02040C2400FCT00/5062453" (id 5) (at 227.33 114.935 0)
+    (property "SUPPLIER_URL" "https://www.digikey.com.au/en/products/detail/vishay-beyschlag-draloric-bc-components/MRS25000C2400FCT00/5064247" (id 5) (at 227.33 114.935 0)
       (effects (font (size 1.27 1.27)) hide)
     )
@@
       (effects (font (size 1.27 1.27)) hide)
     )
-    (property "SUPPLIER_URL" "https://www.digikey.com.au/en/products/detail/vishay-beyschlag-draloric-bc-components/MBA02040C2400FCT00/5062453" (id 4) (at 41.91 36.83 0)
+    (property "SUPPLIER_URL" "https://www.digikey.com.au/en/products/detail/vishay-beyschlag-draloric-bc-components/MRS25000C2400FCT00/5064247" (id 4) (at 41.91 36.83 0)
       (effects (font (size 1.27 1.27)) hide)
     )
@@
     )
     (path "/33a5799b-eb7e-4c0f-a504-681495e3657c"
-      (reference "Q3") (unit 1) (value "SSN1N45") (footprint "Package_TO_SOT_THT:TO-92_Inline_Wide")
+      (reference "Q3") (unit 1) (value "2N7000") (footprint "Package_TO_SOT_THT:TO-92_Inline_Wide")
     )
     (path "/ceb19b93-a3c8-47dc-a451-d369e61f83dc"
@@
     )
     (path "/890c0bff-5da2-4d06-a409-0669cff8cede"
-      (reference "RV1") (unit 1) (value "50k") (footprint "Potentiometer_THT:Potentiometer_Bourns_3296W_Vertical")
+      (reference "RV1") (unit 1) (value "5k") (footprint "Potentiometer_THT:Potentiometer_Bourns_3296W_Vertical")
     )
     (path "/bb6fccf6-b924-49f3-b849-3ed072301c3c"
